Commit message: fix mesh path

File: kuka_kr6r900sixx_description/urdf/kr6r900sixx.urdf (robot description, URDF)
Before this commit: robot kuka_kr6r900sixx, 9 links, 8 joints
Links:
- link base_link: geometry collision mesh filename=package://kuka_kr6r900sixx_description/meshes/collision/bas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; visual mesh filename=package://kuka_kr6r900sixx_description/meshes/visual/base_l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
- link link_1: geometry collision mesh filename=package://kuka_kr6r900sixx_description/meshes/collision/lin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; visual mesh filename=package://kuka_kr6r900sixx_description/meshes/visual/link_1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
- link link_2: geometry collision mesh filename=package://kuka_kr6r900sixx_description/meshes/collision/lin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; visual mesh filename=package://kuka_kr6r900sixx_description/meshes/visual/link_2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
- link link_3: geometry collision mesh filename=package://kuka_kr6r900sixx_description/meshes/collision/lin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; visual mesh filename=package://kuka_kr6r900sixx_description/meshes/visual/link_3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
- link link_4: geometry collision mesh filename=package://kuka_kr6r900sixx_description/meshes/collision/lin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; visual mesh filename=package://kuka_kr6r900sixx_description/meshes/visual/link_4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
- link link_5: geometry collision mesh filename=package://kuka_kr6r900sixx_description/meshes/collision/lin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; visual mesh filename=package://kuka_kr6r900sixx_description/meshes/visual/link_5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
- link link_6: geometry collision mesh filename=package://kuka_kr6r900sixx_description/meshes/collision/lin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; visual mesh filename=package://kuka_kr6r900sixx_description/meshes/visual/link_6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

Commit message: now fix the paths

File: kuka_kr6r900sixx_description/urdf/kr6r900sixx.urdf (robot description, URDF)
Before this commit: robot kuka_kr6r900sixx, 9 links, 8 joints
Links:
- link base_link: geometry collision mesh filename=package://manulab_resources_kuka_kr6r900sixx_description/me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; visual mesh filename=package://manulab_resources_manulab_resources_kuka_kr6r900s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
- link link_1: geometry collision mesh filename=package://manulab_resources_kuka_kr6r900sixx_description/me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; visual mesh filename=package://manulab_resources_kuka_kr6r900sixx_description/me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
- link link_2: geometry collision mesh filename=package://manulab_resources_kuka_kr6r900sixx_description/me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; visual mesh filename=package://manulab_resources_kuka_kr6r900sixx_description/me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
- link link_3: geometry collision mesh filename=package://manulab_resources_kuka_kr6r900sixx_description/me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; visual mesh filename=package://manulab_resources_kuka_kr6r900sixx_description/me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
- link link_4: geometry collision mesh filename=package://manulab_resources_kuka_kr6r900sixx_description/me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; visual mesh filename=package://manulab_resources_kuka_kr6r900sixx_description/me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
- link link_5: geometry collision mesh filename=package://manulab_resources_kuka_kr6r900sixx_description/me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; visual mesh filename=package://manulab_resources_kuka_kr6r900sixx_description/me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
- link link_6: geometry collision mesh filename=package://manulab_resources_kuka_kr6r900sixx_description/me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; visual mesh filename=package://manulab_resources_kuka_kr6r900sixx_description/me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

Commit message: removed erronous search replace

File: kuka_kr6r900sixx_description/urdf/kr6r900sixx.urdf (robot description, URDF)
Before this commit: robot kuka_kr6r900sixx, 9 links, 8 joints
Links:
- link base_link: geometry collision mesh filename=package://manulab_resources_kuka_kr6r900sixx_description/me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; visual mesh filename=package://manulab_resources_kuka_kr6r900sixx_description/me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
