Commit message: support -> description

File: kuka_kr16_description/urdf/kr16.urdf (robot description, URDF)
Before this commit: robot kuka_kr16_2, 9 links, 8 joints
Links:
- link base_link: geometry collision mesh filename=package://kuka_kr16_description/meshes/collision/base_link.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; visual mesh filename=package://kuka_kr16_description/meshes/visual/base_link.dae
- link link_1: geometry collision mesh filename=package://kuka_kr16_description/meshes/collision/link_1.stl; visual mesh filename=package://kuka_kr16_description/meshes/visual/link_1.dae
- link link_2: geometry collision mesh filename=package://kuka_kr16_description/meshes/collision/link_2.stl; visual mesh filename=package://kuka_kr16_description/meshes/visual/link_2.dae
- link link_3: geometry collision mesh filename=package://kuka_kr16_description/meshes/collision/link_3.stl; visual mesh filename=package://kuka_kr16_description/meshes/visual/link_3.dae
- link link_4: geometry collision mesh filename=package://kuka_kr16_description/meshes/collision/link_4.stl; visual mesh filename=package://kuka_kr16_description/meshes/visual/link_4.dae
- link link_5: geometry collision mesh filename=package://kuka_kr16_description/meshes/collision/link_5.stl; visual mesh filename=package://kuka_kr16_description/meshes/visual/link_5.dae
- link link_6: geometry collision mesh filename=package://kuka_kr16_description/meshes/collision/link_6.stl; visual mesh filename=package://kuka_kr16_description/meshes/visual/link_6.dae

Commit message: added manulab_resources prefix

File: kuka_kr16_description/urdf/kr16.urdf (robot description, URDF)
Before this commit: robot kuka_kr16_2, 9 links, 8 joints
Links:
- link base_link: geometry collision mesh filename=package://manulab_resources_kuka_kr16_description/meshes/co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; visual mesh filename=package://manulab_resources_kuka_kr16_description/meshes/vi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
- link link_1: geometry collision mesh filename=package://manulab_resources_kuka_kr16_description/meshes/co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; visual mesh filename=package://manulab_resources_kuka_kr16_description/meshes/vi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
- link link_2: geometry collision mesh filename=package://manulab_resources_kuka_kr16_description/meshes/co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; visual mesh filename=package://manulab_resources_kuka_kr16_description/meshes/vi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
- link link_3: geometry collision mesh filename=package://manulab_resources_kuka_kr16_description/meshes/co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; visual mesh filename=package://manulab_resources_kuka_kr16_description/meshes/vi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
- link link_4: geometry collision mesh filename=package://manulab_resources_kuka_kr16_description/meshes/co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; visual mesh filename=package://manulab_resources_kuka_kr16_description/meshes/vi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
- link link_5: geometry collision mesh filename=package://manulab_resources_kuka_kr16_description/meshes/co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; visual mesh filename=package://manulab_resources_kuka_kr16_description/meshes/vi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
- link link_6: geometry collision mesh filename=package://manulab_resources_kuka_kr16_description/meshes/co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; visual mesh filename=package://manulab_resources_kuka_kr16_description/meshes/vi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
